Commit message: Changed parameters in OMPL planning, changed joint limits in URDF (restricted)

File: movo_common/movo_description/urdf/manipulation/jaco/jaco_7dof.urdf.xacro (robot description, xacro)
@@ -85,5 +85,6 @@
             <origin xyz="0 0 0.0625" rpy="${shoulder_pan_joint_rpy}" />
             <axis xyz="0 0 1" />
-            <limit lower="${-M_PI}" upper="${M_PI}" effort="18000.0" velocity="0.691150384"/>
+            <limit lower="-2.0" upper="1.9" effort="18000.0" velocity="0.691150384"/>
+            <!--<limit lower="${-M_PI}" upper="${M_PI}" effort="18000.0" velocity="0.691150384"/>-->
             <dynamics damping="0.01" friction="0.0"/>
         </joint>
@@ -121,5 +122,6 @@
             <origin xyz="0 0 -0.11875" rpy="${shoulder_lift_joint_rpy}" />
             <axis xyz="0 0 1" />
-            <limit lower="-2.238" upper="2.238" effort="30000.5" velocity="0.691150384"/>
+            <limit lower="-1.5" upper="0.7" effort="30000.5" velocity="0.691150384"/>
+            <!--<limit lower="-2.238" upper="2.238" effort="30000.5" velocity="0.691150384"/>-->
             <dynamics damping="0.01" friction="0.0"/>
         </joint>
@@ -193,5 +195,6 @@
             <origin xyz="0 0 -0.205" rpy="${elbow_joint_rpy}" />
             <axis xyz="0 0 1" />
-            <limit lower="-2.809" upper="2.809" effort="18000.0" velocity="0.691150384"/>
+            <limit lower="-2.6" upper="2.3" effort="18000.0" velocity="0.691150384"/>
+            <!--<limit lower="-2.809" upper="2.809" effort="18000.0" velocity="0.691150384"/>-->
             <dynamics damping="0.01" friction="0.0"/>
         </joint>

Commit message: Adjusted shoulder lift limit

File: movo_common/movo_description/urdf/manipulation/jaco/jaco_7dof.urdf.xacro (robot description, xacro)
@@ -122,5 +122,5 @@
             <origin xyz="0 0 -0.11875" rpy="${shoulder_lift_joint_rpy}" />
             <axis xyz="0 0 1" />
-            <limit lower="-1.5" upper="0.7" effort="30000.5" velocity="0.691150384"/>
+            <limit lower="-1.7" upper="0.7" effort="30000.5" velocity="0.691150384"/>
             <!--<limit lower="-2.238" upper="2.238" effort="30000.5" velocity="0.691150384"/>-->
             <dynamics damping="0.01" friction="0.0"/>

Commit message: Adjust shoulder lift joint limit

File: movo_common/movo_description/urdf/manipulation/jaco/jaco_7dof.urdf.xacro (robot description, xacro)
@@ -122,5 +122,5 @@
             <origin xyz="0 0 -0.11875" rpy="${shoulder_lift_joint_rpy}" />
             <axis xyz="0 0 1" />
-            <limit lower="-1.7" upper="0.7" effort="30000.5" velocity="0.691150384"/>
+            <limit lower="-1.7" upper="1.7" effort="30000.5" velocity="0.691150384"/>
             <!--<limit lower="-2.238" upper="2.238" effort="30000.5" velocity="0.691150384"/>-->
             <dynamics damping="0.01" friction="0.0"/>

Commit message: Modifying OMPL planning as per Panda arm configs, restore joint limits as per original urdf

File: movo_common/movo_description/urdf/manipulation/jaco/jaco_7dof.urdf.xacro (robot description, xacro)
@@ -85,6 +85,6 @@
             <origin xyz="0 0 0.0625" rpy="${shoulder_pan_joint_rpy}" />
             <axis xyz="0 0 1" />
-            <limit lower="-2.0" upper="1.9" effort="18000.0" velocity="0.691150384"/>
-            <!--<limit lower="${-M_PI}" upper="${M_PI}" effort="18000.0" velocity="0.691150384"/>-->
+            <!--<limit lower="-2.0" upper="1.9" effort="18000.0" velocity="0.691150384"/>-->
+            <limit lower="${-M_PI}" upper="${M_PI}" effort="18000.0" velocity="0.691150384"/>
             <dynamics damping="0.01" friction="0.0"/>
         </joint>
@@ -122,6 +122,6 @@
             <origin xyz="0 0 -0.11875" rpy="${shoulder_lift_joint_rpy}" />
             <axis xyz="0 0 1" />
-            <limit lower="-1.7" upper="1.7" effort="30000.5" velocity="0.691150384"/>
-            <!--<limit lower="-2.238" upper="2.238" effort="30000.5" velocity="0.691150384"/>-->
+            <!--<limit lower="-1.7" upper="1.7" effort="30000.5" velocity="0.691150384"/>-->
+            <limit lower="-2.238" upper="2.238" effort="30000.5" velocity="0.691150384"/>
             <dynamics damping="0.01" friction="0.0"/>
         </joint>
@@ -195,6 +195,6 @@
             <origin xyz="0 0 -0.205" rpy="${elbow_joint_rpy}" />
             <axis xyz="0 0 1" />
-            <limit lower="-2.6" upper="2.3" effort="18000.0" velocity="0.691150384"/>
-            <!--<limit lower="-2.809" upper="2.809" effort="18000.0" velocity="0.691150384"/>-->
+            <!--<limit lower="-2.6" upper="2.3" effort="18000.0" velocity="0.691150384"/>-->
+            <limit lower="-2.809" upper="2.809" effort="18000.0" velocity="0.691150384"/>
             <dynamics damping="0.01" friction="0.0"/>
         </joint>
