Commit message: update kinova stuff

File: movo_common/movo_description/urdf/movo_components/movo_pan_tilt.urdf copy.xacro (robot description, xacro)
@@ -133,15 +133,15 @@
 		</link>
 		<xacro:sensor_d435 parent="tilt_link">
-			<origin xyz="0.0699 -0.06 -0.03" rpy="${-M_PI/2} 0 ${-M_PI/2}" />
+			<origin xyz="0.196 -0.06 -0.03" rpy="${-M_PI/2} 0 ${-7*M_PI/12}" />
 		</xacro:sensor_d435>
 		<joint name="tablet_gimbal" type="fixed">
 			<parent link="tilt_link"/>
 			<child link ="tablet_and_mount"/>
-			<origin xyz="0.18515 -0.06 -0.03 " rpy="0 0 ${-M_PI/2}"/>
+			<origin xyz="0.075 -0.06 -0.03 " rpy="0 0 ${-M_PI/2}"/>
 		</joint>
 		<link name="tablet_and_mount" parent="tilt_link">
 			<visual>
 			  <geometry>
-			    <box size="0.02 0.173 0.275"/>
+			    <box size="0.02 0.24 0.3"/>
 		 	  </geometry>
 			  <material name="silver">
@@ -151,5 +151,5 @@
 			<collision>
 			  <geometry>
-			    <box size="0.02 0.173 0.275"/>
+			    <box size="0.04 0.26 0.5"/>
 		 	  </geometry>
 			</collision>
@@ -158,10 +158,10 @@
 			<parent link="tilt_link"/>
 			<child link ="mating_block"/>
-			<origin xyz="0.14 0 -0.03 " rpy="0 0 0"/>
+			<origin xyz="0.09 0 -0.03 " rpy="0 0 0"/>
 		</joint>
 		<link name="mating_block" parent="tilt_link">
 			<visual>
 			  <geometry>
-			    <box size="0.166 0.066 0.13"/>
+			    <box size="0.066 0.066 0.13"/>
 		 	  </geometry>
 			  <material name="silver"/>
@@ -169,9 +169,9 @@
 			<collision>
 			  <geometry>
-			    <box size="0.166 0.066 0.13"/>
+			    <box size="0.084 0.084 0.13"/>
 		 	  </geometry>
 			</collision>
 		</link>
-		<!-- <joint name="camera_mount_gimbal" type="fixed">
+		<joint name="camera_mount_gimbal" type="fixed">
 			<parent link="tilt_link"/>
 			<child link ="camera_mount"/>
@@ -190,5 +190,5 @@
 		 	  </geometry>
 			</collision>
-		</link> -->
+		</link>
     </xacro:macro>
 </robot>
